File: mrmeeseeks.sch (KiCad schematic (older format))
At the start: 34 parts

Commit message: Schematic Complete
Parts:
- removed U?: ATTINY85-20PU, Housings_DIP:DIP-8_W7.62mm, symbol ATTINY85-20PU
- added C1: 0.1uf, Capacitors_SMD:C_0402_NoSilk, symbol C
- D1, D10, D11, D12, D13, D14, D15, D16, D2, D3, D4, D5, D6, D7, D8, D9: renamed from D?; footprint (none) -> LEDs:LED_1206_HandSoldering
- R1, R10, R11, R12, R13, R14, R15, R16, R2, R3, R4, R5, R6, R7, R8, R9: renamed from R?; footprint (none) -> Resistors_SMD:R_1206_HandSoldering
- U1: renamed from U?; footprint (none) -> SMD_Packages:SOIC-28
Connections:
- net +3V3: now also U1.18 (~RESET), U1.9 (VCC), C1.1
- net GND: now reaches U1.10 (GND)
- net GND: now also D1.1 (K), D10.1 (K), D11.1 (K), D12.1 (K), D13.1 (K), D14.1 (K), D15.1 (K), D16.1 (K), D2.1 (K), D3.1 (K), D4.1 (K), D5.1 (K), D6.1 (K), D7.1 (K), D8.1 (K), D9.1 (K), U1.15 (A0), U1.16 (A1), U1.17 (A2), C1.2
- net scl: now reaches U1.12 (SCL)
- net sda: now reaches U1.13 (SDA)

Commit message: Updated PCB Design
Parts:
- removed D10, D11, D12, D13, D14, D15, D16: LED, LEDs:LED_1206_HandSoldering, symbol LED
- removed R10, R11, R12, R13, R14, R15, R16: 220, Resistors_SMD:R_1206_HandSoldering, symbol R
- added X1: Badgelife_shitty_connector, mrmeeseeks-addon:Badgelife-Shitty-2x2, symbol Badgelife_shitty_connector
Connections:
- wire segments 54 -> 40
