File: mrmeeseeks.kicad_pcb (KiCad board)
At the start: 2 copper layers, 49.6 x 62.4 mm, 23 parts, among them U1 MCP23017, X1 Badgelife_shitty_connector

Commit message: Revision Tagging
Other:
- board text added: "Designed By: d4rkwyng SparX"
- board text added: "Mr Meeseeks Rev. A"
- board text removed: "Designed By: MyndFyre SparX"
Changed lines of the file:
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@@
     (area 58.674 59.563 148.361401 132.249896)
     (thickness 1.6)
-    (drawings 260)
+    (drawings 261)
     (tracks 223)
     (zones 0)
@@
       (net 31 "Net-(U1-Pad28)"))
   )
+  (gr_text "Mr Meeseeks\nRev. A" (at 99.187 126.5174) (layer B.SilkS)
+    (effects (font (size 0.5 0.5) (thickness 0.125)) (justify mirror))
+  )
   (gr_text "ILLEGAL TO SELL\nON EBAY" (at 98.9584 90.2462) (layer B.SilkS)
     (effects (font (size 2.5 2.5) (thickness 0.3)) (justify mirror))
@@
     (effects (font (size 0.75 0.75) (thickness 0.1)) (justify mirror))
   )
-  (gr_text "Designed By:\nMyndFyre\nSparX" (at 85.27288 113.9952) (layer B.SilkS)
+  (gr_text "Designed By:\nd4rkwyng\nSparX" (at 85.27288 113.9952) (layer B.SilkS)
     (effects (font (size 1 1) (thickness 0.1)) (justify mirror))
   )
