File: mrmeeseeks_RevC.kicad_pcb (KiCad board)
At the start: 2 copper layers, 49.6 x 62.4 mm, 23 parts, among them U1 MCP23017, X1 Badgelife_shitty_connector

Commit message: Revision Tagging
Other:
- board text added: "Mr Meeseeks Rev. C"
Changed lines of the file:
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@@
     (area 74.194599 65.253799 123.976201 127.837001)
     (thickness 1.6)
-    (drawings 260)
+    (drawings 261)
     (tracks 290)
     (zones 0)
@@
   )
   (setup
-    (last_trace_width 0.2)
+    (last_trace_width 0.25)
     (user_trace_width 0.2)
     (user_trace_width 0.5)
@@
       (net 31 "Net-(U1-Pad28)"))
   )
+  (gr_text "Mr Meeseeks\nRev. C" (at 99.1997 126.0094) (layer B.SilkS)
+    (effects (font (size 0.5 0.5) (thickness 0.125)) (justify mirror))
+  )
   (gr_text "ILLEGAL TO SELL\nON EBAY" (at 98.9584 90.2462) (layer B.SilkS)
