File: mrmeeseeks_RevD.kicad_pcb (KiCad board)
At the start: 2 copper layers, 49.6 x 62.4 mm, 23 parts, among them U1 MCP23017, X1 Badgelife_shitty_connector

Commit message: Clean Up
Other:
- board text added: "Designed By: d4rkw1ng SparX"
- board text removed: "Designed By: MyndFyre SparX"
Changed lines of the file:
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@@
   )
   (setup
-    (last_trace_width 0.2)
+    (last_trace_width 0.25)
     (user_trace_width 0.2)
     (user_trace_width 0.5)
@@
     (effects (font (size 1.5 1.5) (thickness 0.3)) (justify mirror))
   )
-  (gr_text "Thanks to:\nAND!XOR" (at 85.344 119.126) (layer B.SilkS)
+  (gr_text "Thanks to:\nAND!XOR" (at 92.47124 122.26544) (layer B.SilkS)
     (effects (font (size 0.75 0.75) (thickness 0.1)) (justify mirror))
   )
-  (gr_text "Designed By:\nMyndFyre\nSparX" (at 106.299 115.824) (layer B.SilkS)
+  (gr_text "Designed By:\nd4rkw1ng\nSparX" (at 106.299 115.824) (layer B.SilkS)
     (effects (font (size 1 1) (thickness 0.1)) (justify mirror))
   )

Commit message: Rev D Updates
Other:
- board text added: "Look at me!"
Changed lines of the file:
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@@
     (area 74.194599 65.253799 123.976201 127.837001)
     (thickness 1.6)
-    (drawings 259)
+    (drawings 260)
     (tracks 173)
     (zones 0)
@@
       (net 31 "Net-(U1-Pad28)"))
   )
+  (gr_text "Look at me!" (at 88.12276 109.07776) (layer B.SilkS)
+    (effects (font (size 1 1) (thickness 0.25)) (justify mirror))
+  )
   (gr_text "Mr Meeseeks\nRev. D" (at 99.441 126.365) (layer B.SilkS)

Commit message: Rev D Updates
Other:
- board text added: "Designed By: d4rkwyng SparX"
- board text removed: "Designed By: d4rkw1ng SparX"
Changed lines of the file:
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@@
     (effects (font (size 0.75 0.75) (thickness 0.1)) (justify mirror))
   )
-  (gr_text "Designed By:\nd4rkw1ng\nSparX" (at 106.299 115.824) (layer B.SilkS)
+  (gr_text "Designed By:\nd4rkwyng\nSparX" (at 106.299 115.824) (layer B.SilkS)
     (effects (font (size 1 1) (thickness 0.1)) (justify mirror))
   )
