File: mrmeeseeks_RevE.kicad_pcb (KiCad board)
At the start: 2 copper layers, 49.6 x 62.4 mm, 21 parts, among them U1 MCP23017, X1 Badgelife_shitty_connector

Commit message: Show Me What You've Got Update
Parts:
- added G***: LOGO, mrmeeseeks-design:smwyg, B.Cu at (109.2, 113.8)

Commit message: The terror that flaps in the night!
Parts:
- added G***: LOGO, mrmeeseeks-design:d4rkwyng, B.Cu at (89.9, 112.8)
- added G***: LOGO, mrmeeseeks-design:d4rkwyng_solder, B.Cu at (89.9, 112.8)
- moved G*** 2.16 mm to (110.7, 112.3)

Commit message: Minor Library Changes
Parts:
- U1: footprint INTERFACE-MCP23017-E_SOIC28_:SOIC28-1.27-17.9X7.5MM -> mrmeeseeks-lib:MCP23017-ESO_NoSilk
Changed lines of the file:
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@@
     (links 34)
     (no_connects 0)
-    (area 74.194599 65.253799 123.976201 127.837001)
+    (area 58.674 59.563 148.361401 132.249896)
     (thickness 1.6)
     (drawings 260)
@@
     )
   )
-  (module INTERFACE-MCP23017-E_SOIC28_:SOIC28-1.27-17.9X7.5MM (layer B.Cu)
-    (at 98.96348 100.7237)
-    (attr smd)
-    (fp_text reference U1 (at -10.0068 -0.127481 90) (layer F.Fab)
-      (effects (font (size 0.702618 0.702618) (thickness 0.05)))
-    )
-    (fp_text value MCP23017 (at -2.35561 0.318324 270) (layer B.SilkS)
-      (effects (font (size 0.701821 0.701821) (thickness 0.05)) (justify mirror))
-    )
-    (fp_line (start -8.95 3.75) (end -8.95 -2.84797) (layer B.SilkS) (width 0.1524))
-    (fp_line (start -8.95 -2.84797) (end -8.04797 -3.75) (layer B.SilkS) (width 0.1524))
-    (fp_line (start -8.04797 -3.75) (end 8.95 -3.75) (layer B.SilkS) (width 0.1524))
-    (fp_line (start 8.95 -3.75) (end 8.95 3.75) (layer B.SilkS) (width 0.1524))
-    (fp_line (start 8.95 3.75) (end -8.95 3.75) (layer B.SilkS) (width 0.1524))
-    (fp_circle (center -9.275 -4.175) (end -8.894 -4.175) (layer B.SilkS) (width 0))
-    (fp_poly (pts (xy -8.97374 3.658) (xy 8.95 3.658) (xy 8.95 -3.69277) (xy -8.97374 -3.69277)) (layer Dwgs.User) (width 0.381))
-    (pad 1 smd rect (at -8.255 -4.7498) (size 0.762 1.143) (layers B.Cu B.Paste B.Mask)
-      (net 11 "Net-(R1-Pad1)"))
-    (pad 2 smd rect (at -6.985 -4.7498) (size 0.762 1.143) (layers B.Cu B.Paste B.Mask)
-      (net 12 "Net-(R2-Pad1)"))
-    (pad 3 smd rect (at -5.715 -4.7498) (size 0.762 1.143) (layers B.Cu B.Paste B.Mask)
-      (net 13 "Net-(R3-Pad1)"))
-    (pad 4 smd rect (at -4.445 -4.7498) (size 0.762 1.143) (layers B.Cu B.Paste B.Mask)
-      (net 14 "Net-(R4-Pad1)"))
-    (pad 5 smd rect (at -3.175 -4.7498) (size 0.762 1.143) (layers B.Cu B.Paste B.Mask)
-      (net 15 "Net-(R5-Pad1)"))
-    (pad 6 smd rect (at -1.905 -4.7498) (size 0.762 1.143) (layers B.Cu B.Paste B.Mask)
-      (net 16 "Net-(R6-Pad1)"))
-    (pad 7 smd rect (at -0.635 -4.7498) (size 0.762 1.143) (layers B.Cu B.Paste B.Mask)
-      (net 17 "Net-(R7-Pad1)"))
-    (pad 8 smd rect (at 0.635 -4.7498) (size 0.762 1.143) (layers B.Cu B.Paste B.Mask)
-      (net 18 "Net-(R8-Pad1)"))
-    (pad 9 smd rect (at 1.905 -4.7498) (size 0.762 1.143) (layers B.Cu B.Paste B.Mask)
-      (net 1 +3V3))
-    (pad 10 smd rect (at 3.175 -4.7498) (size 0.762 1.143) (layers B.Cu B.Paste B.Mask)
-      (net 2 GND))
-    (pad 12 smd rect (at 5.715 -4.7498) (size 0.762 1.143) (layers B.Cu B.Paste B.Mask)
-      (net 20 scl))
-    (pad 11 smd rect (at 4.445 -4.7498) (size 0.762 1.143) (layers B.Cu B.Paste B.Mask))
-    (pad 13 smd rect (at 6.985 -4.7498) (size 0.762 1.143) (layers B.Cu B.Paste B.Mask)
-      (net 21 sda))
-    (pad 14 smd rect (at 8.255 -4.7498) (size 0.762 1.143) (layers B.Cu B.Paste B.Mask))
-    (pad 15 smd rect (at 8.255 4.7752) (size 0.762 1.143) (layers B.Cu B.Paste B.Mask)
-      (net 2 GND))
-    (pad 16 smd rect (at 6.985 4.7752) (size 0.762 1.143) (layers B.Cu B.Paste B.Mask)
-      (net 2 GND))
-    (pad 17 smd rect (at 5.715 4.7752) (size 0.762 1.143) (layers B.Cu B.Paste B.Mask)
-      (net 2 GND))
-    (pad 18 smd rect (at 4.445 4.7752) (size 0.762 1.143) (layers B.Cu B.Paste B.Mask)
-      (net 1 +3V3))
-    (pad 19 smd rect (at 3.175 4.7752) (size 0.762 1.143) (layers B.Cu B.Paste B.Mask)
-      (net 22 "Net-(U1-Pad19)"))
-    (pad 20 smd rect (at 1.905 4.7752) (size 0.762 1.143) (layers B.Cu B.Paste B.Mask)
-      (net 23 "Net-(U1-Pad20)"))
-    (pad 21 smd rect (at 0.635 4.7752) (size 0.762 1.143) (layers B.Cu B.Paste B.Mask)
-      (net 19 "Net-(R9-Pad1)"))
-    (pad 22 smd rect (at -0.635 4.7752) (size 0.762 1.143) (layers B.Cu B.Paste B.Mask)
-      (net 24 "Net-(U1-Pad22)"))
-    (pad 23 smd rect (at -1.905 4.7752) (size 0.762 1.143) (layers B.Cu B.Paste B.Mask)
-      (net 25 "Net-(U1-Pad23)"))
-    (pad 24 smd rect (at -3.175 4.7752) (size 0.762 1.143) (layers B.Cu B.Paste B.Mask)
-      (net 26 "Net-(U1-Pad24)"))
-    (pad 25 smd rect (at -4.445 4.7752) (size 0.762 1.143) (layers B.Cu B.Paste B.Mask)
-      (net 27 "Net-(U1-Pad25)"))
-    (pad 26 smd rect (at -5.715 4.7752) (size 0.762 1.143) (layers B.Cu B.Paste B.Mask)
-      (net 28 "Net-(U1-Pad26)"))
-    (pad 27 smd rect (at -6.985 4.7752) (size 0.762 1.143) (layers B.Cu B.Paste B.Mask)
-      (net 29 "Net-(U1-Pad27)"))
-    (pad 28 smd rect (at -8.255 4.7752) (size 0.762 1.143) (layers B.Cu B.Paste B.Mask)
-      (net 30 "Net-(U1-Pad28)"))
-  )
   (module Capacitors_SMD:C_1206_HandSoldering (layer B.Cu)
     (at 84.7344 101.9175 270)
@@
       (xy -0.0244 -0.348367) (xy 0.000409 -0.344503) (xy 0.007379 -0.34733)) (layer B.Mask) (width 0.01))
   )
+  (module mrmeeseeks-lib:MCP23017-ESO_NoSilk (layer B.Cu)
+    (at 98.96348 100.7237)
+    (attr smd)
+    (fp_text reference U1 (at -10.0068 -0.127481 270) (layer B.Fab)
+      (effects (font (size 0.702618 0.702618) (thickness 0.05)) (justify mirror))
+    )
+    (fp_text value MCP23017 (at -2.35561 0.318324) (layer B.Fab)
+      (effects (font (size 0.701821 0.701821) (thickness 0.05)) (justify mirror))
+    )
+    (fp_line (start -8.95 3.75) (end -8.95 -2.84797) (layer B.SilkS) (width 0.1524))
+    (fp_line (start -8.95 -2.84797) (end -8.04797 -3.75) (layer B.SilkS) (width 0.1524))
+    (fp_line (start -8.04797 -3.75) (end 8.95 -3.75) (layer B.SilkS) (width 0.1524))
+    (fp_line (start 8.95 -3.75) (end 8.95 3.75) (layer B.SilkS) (width 0.1524))
+    (fp_line (start 8.95 3.75) (end -8.95 3.75) (layer B.SilkS) (width 0.1524))
+    (fp_circle (center -9.275 -4.175) (end -8.894 -4.175) (layer B.SilkS) (width 0))
+    (fp_poly (pts (xy -8.97374 3.658) (xy 8.95 3.658) (xy 8.95 -3.69277) (xy -8.97374 -3.69277)) (layer Dwgs.User) (width 0.381))
+    (pad 1 smd rect (at -8.255 -4.7498) (size 0.762 1.143) (layers B.Cu B.Paste B.Mask)
+      (net 11 "Net-(R1-Pad1)"))
+    (pad 2 smd rect (at -6.985 -4.7498) (size 0.762 1.143) (layers B.Cu B.Paste B.Mask)
+      (net 12 "Net-(R2-Pad1)"))
+    (pad 3 smd rect (at -5.715 -4.7498) (size 0.762 1.143) (layers B.Cu B.Paste B.Mask)
+      (net 13 "Net-(R3-Pad1)"))
+    (pad 4 smd rect (at -4.445 -4.7498) (size 0.762 1.143) (layers B.Cu B.Paste B.Mask)
+      (net 14 "Net-(R4-Pad1)"))
+    (pad 5 smd rect (at -3.175 -4.7498) (size 0.762 1.143) (layers B.Cu B.Paste B.Mask)
+      (net 15 "Net-(R5-Pad1)"))
+    (pad 6 smd rect (at -1.905 -4.7498) (size 0.762 1.143) (layers B.Cu B.Paste B.Mask)
+      (net 16 "Net-(R6-Pad1)"))
+    (pad 7 smd rect (at -0.635 -4.7498) (size 0.762 1.143) (layers B.Cu B.Paste B.Mask)
+      (net 17 "Net-(R7-Pad1)"))
+    (pad 8 smd rect (at 0.635 -4.7498) (size 0.762 1.143) (layers B.Cu B.Paste B.Mask)
+      (net 18 "Net-(R8-Pad1)"))
+    (pad 9 smd rect (at 1.905 -4.7498) (size 0.762 1.143) (layers B.Cu B.Paste B.Mask)
+      (net 1 +3V3))
+    (pad 10 smd rect (at 3.175 -4.7498) (size 0.762 1.143) (layers B.Cu B.Paste B.Mask)
+      (net 2 GND))
+    (pad 12 smd rect (at 5.715 -4.7498) (size 0.762 1.143) (layers B.Cu B.Paste B.Mask)
+      (net 20 scl))
+    (pad 11 smd rect (at 4.445 -4.7498) (size 0.762 1.143) (layers B.Cu B.Paste B.Mask))
+    (pad 13 smd rect (at 6.985 -4.7498) (size 0.762 1.143) (layers B.Cu B.Paste B.Mask)
+      (net 21 sda))
+    (pad 14 smd rect (at 8.255 -4.7498) (size 0.762 1.143) (layers B.Cu B.Paste B.Mask))
+    (pad 15 smd rect (at 8.255 4.7752) (size 0.762 1.143) (layers B.Cu B.Paste B.Mask)
+      (net 2 GND))
+    (pad 16 smd rect (at 6.985 4.7752) (size 0.762 1.143) (layers B.Cu B.Paste B.Mask)
+      (net 2 GND))
+    (pad 17 smd rect (at 5.715 4.7752) (size 0.762 1.143) (layers B.Cu B.Paste B.Mask)
+      (net 2 GND))
+    (pad 18 smd rect (at 4.445 4.7752) (size 0.762 1.143) (layers B.Cu B.Paste B.Mask)
+      (net 1 +3V3))
+    (pad 19 smd rect (at 3.175 4.7752) (size 0.762 1.143) (layers B.Cu B.Paste B.Mask)
+      (net 22 "Net-(U1-Pad19)"))
+    (pad 20 smd rect (at 1.905 4.7752) (size 0.762 1.143) (layers B.Cu B.Paste B.Mask)
+      (net 23 "Net-(U1-Pad20)"))
+    (pad 21 smd rect (at 0.635 4.7752) (size 0.762 1.143) (layers B.Cu B.Paste B.Mask)
+      (net 19 "Net-(R9-Pad1)"))
+    (pad 22 smd rect (at -0.635 4.7752) (size 0.762 1.143) (layers B.Cu B.Paste B.Mask)
+      (net 24 "Net-(U1-Pad22)"))
+    (pad 23 smd rect (at -1.905 4.7752) (size 0.762 1.143) (layers B.Cu B.Paste B.Mask)
+      (net 25 "Net-(U1-Pad23)"))
+    (pad 24 smd rect (at -3.175 4.7752) (size 0.762 1.143) (layers B.Cu B.Paste B.Mask)
+      (net 26 "Net-(U1-Pad24)"))
+    (pad 25 smd rect (at -4.445 4.7752) (size 0.762 1.143) (layers B.Cu B.Paste B.Mask)
+      (net 27 "Net-(U1-Pad25)"))
+    (pad 26 smd rect (at -5.715 4.7752) (size 0.762 1.143) (layers B.Cu B.Paste B.Mask)
+      (net 28 "Net-(U1-Pad26)"))
+    (pad 27 smd rect (at -6.985 4.7752) (size 0.762 1.143) (layers B.Cu B.Paste B.Mask)
+      (net 29 "Net-(U1-Pad27)"))
+    (pad 28 smd rect (at -8.255 4.7752) (size 0.762 1.143) (layers B.Cu B.Paste B.Mask)
+      (net 30 "Net-(U1-Pad28)"))
+  )
   (gr_text "Look at me!" (at 85.344 93.98) (layer B.SilkS)
