File: mrmeeseeks_RevE.sch (KiCad schematic (older format))
At the start: 19 parts, among them U1 MCP23017, X1 Badgelife_shitty_connector

Commit message: Finish footprint library cleanup left incomplete by d13783b
d13783b fixed the RevE schematic's symbol-library ref but the
footprint-library side of the same regression was still broken:
fp-lib-table only declared mrmeeseeks-design, while every populated
footprint on the RevE/RevE_ESO boards (U1, X1, R1-R8, D1-D8) actually
uses the mrmeeseeks-addon, mrmeeseeks-addon-design or mrmeeseeks-lib
nicknames, none of which had table entries. Confirmed with
`kicad-cli pcb drc`: RevE dropped from 21 lib_footprint_issues to 1
(the sole remainder, Capacitors_SMD, is KiCad's own stock library and
out of repo scope); RevA-D pick up the mrmeeseeks-addon-design entry
too.

- fp-lib-table: add mrmeeseeks-addon-design, mrmeeseeks-addon,
  mrmeeseeks-lib, all pointing at their real directories (design/, lib/).
- design/mrmeeseeks-silkscreen.kicad_mod -> design/silkscreen.kicad_mod
  and mrmeeseeks-soldermask.kicad_mod -> soldermask.kicad_mod: KiCad's
  directory-type footprint libraries resolve by filename, not the
  internal (module NAME ...) field, so these never matched what the
  boards call mrmeeseeks-design:silkscreen / mrmeeseeks-addon-design:soldermask.
- mrmeeseeks_RevE.pro: LastNetListRead=mrmeeseeksRevE.net was missing
  the underscore the actual mrmeeseeks_RevE.net file has -- same
  Rev-E-rename regression class d13783b fixed in the schematic header.
- mrmeeseeks_RevE.sch: corrected 17 stale F2 footprint-assignment
  fields (D1-D8, R1-R8, X1) that pointed at generic/nonexistent
  libraries (LEDs, Resistors_SMD, lib) instead of the mrmeeseeks-addon
  footprints actually placed on the board and listed in
  mrmeeseeks_RevE_BOM.csv. Left U1's field cleared rather than guessing
  ESO vs ESS, since this one schematic backs both mrmeeseeks_RevE.kicad_pcb
  (MCP23017-ESO_NoSilk) and mrmeeseeks_RevE_ESO.kicad_pcb (confusingly,
  MCP23017-ESS_NoSilk) -- open question for Derek below.

Co-Authored-By: Claude Sonnet 5 <noreply@anthropic.com>
Parts:
- D1, D2, D3, D4, D5, D6, D7, D8: footprint LEDs:LED_1206_HandSoldering -> mrmeeseeks-addon:LED_1206_HandSoldering_MinSilk
- R1, R2, R3, R4, R5, R6, R7, R8: footprint Resistors_SMD:R_1206_HandSoldering -> mrmeeseeks-addon:R_1206_HandSoldering_NoSilk
- U1: footprint INTERFACE-MCP23017-E_SOIC28_:SOIC28-1.27-17.9X7.5MM -> (none)
- X1: footprint lib:Badgelife-Shitty-2x2 -> mrmeeseeks-addon:Badgelife-Shitty-2x2
Changed lines of the file:
@@
 F 0 "U1" H 3950 4375 50  0000 R CNN
 F 1 "MCP23017" H 3950 4300 50  0000 R CNN
-F 2 "INTERFACE-MCP23017-E_SOIC28_:SOIC28-1.27-17.9X7.5MM" H 4100 2400 50  0001 L CNN
+F 2 "" H 4100 2400 50  0001 L CNN
 F 3 "" H 4300 4350 50  0001 C CNN
 	1    4050 3350
@@
 F 0 "D1" H 2800 2650 50  0000 C CNN
 F 1 "LED" H 2800 2450 50  0000 C CNN
-F 2 "LEDs:LED_1206_HandSoldering" H 2800 2550 50  0001 C CNN
+F 2 "mrmeeseeks-addon:LED_1206_HandSoldering_MinSilk" H 2800 2550 50  0001 C CNN
 F 3 "" H 2800 2550 50  0001 C CNN
 	1    2800 2550
@@
 F 0 "D2" H 2800 2750 50  0000 C CNN
 F 1 "LED" H 2800 2550 50  0000 C CNN
-F 2 "LEDs:LED_1206_HandSoldering" H 2800 2650 50  0001 C CNN
+F 2 "mrmeeseeks-addon:LED_1206_HandSoldering_MinSilk" H 2800 2650 50  0001 C CNN
 F 3 "" H 2800 2650 50  0001 C CNN
 	1    2800 2650
@@
 F 0 "D3" H 2800 2850 50  0000 C CNN
 F 1 "LED" H 2800 2650 50  0000 C CNN
-F 2 "LEDs:LED_1206_HandSoldering" H 2800 2750 50  0001 C CNN
+F 2 "mrmeeseeks-addon:LED_1206_HandSoldering_MinSilk" H 2800 2750 50  0001 C CNN
 F 3 "" H 2800 2750 50  0001 C CNN
 	1    2800 2750
@@
 F 0 "D4" H 2800 2950 50  0000 C CNN
 F 1 "LED" H 2800 2750 50  0000 C CNN
-F 2 "LEDs:LED_1206_HandSoldering" H 2800 2850 50  0001 C CNN
+F 2 "mrmeeseeks-addon:LED_1206_HandSoldering_MinSilk" H 2800 2850 50  0001 C CNN
 F 3 "" H 2800 2850 50  0001 C CNN
 	1    2800 2850
@@
 F 0 "D5" H 2800 3050 50  0000 C CNN
 F 1 "LED" H 2800 2850 50  0000 C CNN
-F 2 "LEDs:LED_1206_HandSoldering" H 2800 2950 50  0001 C CNN
+F 2 "mrmeeseeks-addon:LED_1206_HandSoldering_MinSilk" H 2800 2950 50  0001 C CNN
 F 3 "" H 2800 2950 50  0001 C CNN
 	1    2800 2950
@@
 F 0 "D6" H 2800 3150 50  0000 C CNN
 F 1 "LED" H 2800 2950 50  0000 C CNN
-F 2 "LEDs:LED_1206_HandSoldering" H 2800 3050 50  0001 C CNN
+F 2 "mrmeeseeks-addon:LED_1206_HandSoldering_MinSilk" H 2800 3050 50  0001 C CNN
 F 3 "" H 2800 3050 50  0001 C CNN
 	1    2800 3050
@@
 F 0 "D7" H 2800 3250 50  0000 C CNN
 F 1 "LED" H 2800 3050 50  0000 C CNN
-F 2 "LEDs:LED_1206_HandSoldering" H 2800 3150 50  0001 C CNN
+F 2 "mrmeeseeks-addon:LED_1206_HandSoldering_MinSilk" H 2800 3150 50  0001 C CNN
 F 3 "" H 2800 3150 50  0001 C CNN
 	1    2800 3150
@@
 F 0 "D8" H 2800 3350 50  0000 C CNN
 F 1 "LED" H 2800 3150 50  0000 C CNN
-F 2 "LEDs:LED_1206_HandSoldering" H 2800 3250 50  0001 C CNN
+F 2 "mrmeeseeks-addon:LED_1206_HandSoldering_MinSilk" H 2800 3250 50  0001 C CNN
 F 3 "" H 2800 3250 50  0001 C CNN
 	1    2800 3250
@@
 F 0 "R1" V 3330 2550 50  0000 C CNN
 F 1 "220" V 3250 2550 50  0000 C CNN
-F 2 "Resistors_SMD:R_1206_HandSoldering" V 3180 2550 50  0001 C CNN
+F 2 "mrmeeseeks-addon:R_1206_HandSoldering_NoSilk" V 3180 2550 50  0001 C CNN
 F 3 "" H 3250 2550 50  0001 C CNN
 	1    3250 2550
@@
 F 0 "R2" V 3330 2650 50  0000 C CNN
 F 1 "220" V 3250 2650 50  0000 C CNN
-F 2 "Resistors_SMD:R_1206_HandSoldering" V 3180 2650 50  0001 C CNN
+F 2 "mrmeeseeks-addon:R_1206_HandSoldering_NoSilk" V 3180 2650 50  0001 C CNN
 F 3 "" H 3250 2650 50  0001 C CNN
 	1    3250 2650
@@
 F 0 "R3" V 3330 2750 50  0000 C CNN
 F 1 "220" V 3250 2750 50  0000 C CNN
-F 2 "Resistors_SMD:R_1206_HandSoldering" V 3180 2750 50  0001 C CNN
+F 2 "mrmeeseeks-addon:R_1206_HandSoldering_NoSilk" V 3180 2750 50  0001 C CNN
 F 3 "" H 3250 2750 50  0001 C CNN
 	1    3250 2750
@@
 F 0 "R4" V 3330 2850 50  0000 C CNN
 F 1 "220" V 3250 2850 50  0000 C CNN
-F 2 "Resistors_SMD:R_1206_HandSoldering" V 3180 2850 50  0001 C CNN
+F 2 "mrmeeseeks-addon:R_1206_HandSoldering_NoSilk" V 3180 2850 50  0001 C CNN
 F 3 "" H 3250 2850 50  0001 C CNN
 	1    3250 2850
@@
 F 0 "R5" V 3330 2950 50  0000 C CNN
 F 1 "220" V 3250 2950 50  0000 C CNN
-F 2 "Resistors_SMD:R_1206_HandSoldering" V 3180 2950 50  0001 C CNN
+F 2 "mrmeeseeks-addon:R_1206_HandSoldering_NoSilk" V 3180 2950 50  0001 C CNN
 F 3 "" H 3250 2950 50  0001 C CNN
 	1    3250 2950
@@
 F 0 "R6" V 3330 3050 50  0000 C CNN
 F 1 "220" V 3250 3050 50  0000 C CNN
-F 2 "Resistors_SMD:R_1206_HandSoldering" V 3180 3050 50  0001 C CNN
+F 2 "mrmeeseeks-addon:R_1206_HandSoldering_NoSilk" V 3180 3050 50  0001 C CNN
 F 3 "" H 3250 3050 50  0001 C CNN
 	1    3250 3050
@@
 F 0 "R7" V 3330 3150 50  0000 C CNN
 F 1 "220" V 3250 3150 50  0000 C CNN
-F 2 "Resistors_SMD:R_1206_HandSoldering" V 3180 3150 50  0001 C CNN
+F 2 "mrmeeseeks-addon:R_1206_HandSoldering_NoSilk" V 3180 3150 50  0001 C CNN
 F 3 "" H 3250 3150 50  0001 C CNN
 	1    3250 3150
@@
 F 0 "R8" V 3330 3250 50  0000 C CNN
 F 1 "220" V 3250 3250 50  0000 C CNN
-F 2 "Resistors_SMD:R_1206_HandSoldering" V 3180 3250 50  0001 C CNN
+F 2 "mrmeeseeks-addon:R_1206_HandSoldering_NoSilk" V 3180 3250 50  0001 C CNN
 F 3 "" H 3250 3250 50  0001 C CNN
 	1    3250 3250
@@
 F 0 "X1" H 5100 5500 60  0000 C CNN
 F 1 "Badgelife_shitty_connector" H 5000 6100 60  0000 C CNN
-F 2 "lib:Badgelife-Shitty-2x2" H 5000 5700 60  0001 C CNN
+F 2 "mrmeeseeks-addon:Badgelife-Shitty-2x2" H 5000 5700 60  0001 C CNN
 F 3 "" H 5000 5700 60  0001 C CNN
 	1    5000 5700
